Commit message: cartesian: use flange (tool0) as effector frame, not the fingertip
Move the cartesian effector reference from the +0.158m fingertip to the wrist
flange, so per-step position deltas don't pick up the wrist-rotation lever (a
long offset turns small orientation changes into large translations).

- URDF: tool0 is now the FLANGE — link6-7 origin (wrist) with the OpenCV
  orientation (z=approach/front, x=right), matching DROID's panda_link8 choice.
  The old +0.158m fingertip frame is renamed `tcp` (kept for grasp/IK use).
  tool0 = flange is the ROS-Industrial convention; this intentionally DIVERGES
  from the fastwam URDF, where tool0 is the fingertip.
- compute_cartesian.py: FK now uses the default tool0 (= flange).
- Regenerated dk1_action_normalization_cartesian.json: x/y position-delta
  quantiles tightened ~20-25% (lever artifact removed); z (approach) and the
  rot6d block are unchanged (orientation is identical to the old tool0).

Confirms the paper's action spec (single-step SE(3) deltas, 6D rotation, OpenCV
effector frame z=fingers/x=right, absolute grasp state). Caches regenerable via
scripts/compute_cartesian.py (gitignored).

Co-Authored-By: Claude Opus 4.8 <noreply@anthropic.com>

File: urdf/dk1_dual_arm.urdf (robot description, URDF)
Before this commit: robot dk1_dual_arm, 26 links, 25 joints
Links:
- added link left_tcp
- added link right_tcp
Joints:
- added joint left_tcp_joint: type fixed, parent left_link6-7, child left_tcp, origin xyz=0.158 0 0 rpy=-1.5707963267948966 0 -1.5707963267948966
- added joint right_tcp_joint: type fixed, parent right_link6-7, child right_tcp, origin xyz=0.158 0 0 rpy=-1.5707963267948966 0 -1.5707963267948966
- joint left_gripper_tool0: origin xyz=0.158 0 0 rpy=-1.5707963267948966 0 -1.5707963267948966 -> xyz=0 0 0 rpy=-1.5707963267948966 0 -1.5707963267948966
- joint right_gripper_tool0: origin xyz=0.158 0 0 rpy=-1.5707963267948966 0 -1.5707963267948966 -> xyz=0 0 0 rpy=-1.5707963267948966 0 -1.5707963267948966

Commit message: urdf: sync vendored dk1_dual_arm.urdf to upstream dk1-dual-arm-urdf
The upstream URDF already defines exactly the convention we'd hand-edited:
tool0 = flange (link6-7 origin, OpenCV orientation z=front/x=right) and tcp =
the +0.158m fingertip. Replace our hand-edited fork with the upstream file
verbatim — canonical source, cleaner {left,right}_tool0_joint names, and drops
a stale "grip_center" comment.

Geometry is byte-identical to our edited copy (FK matches the existing caches to
~1e-7), so the cartesian caches/stats are unaffected — no regeneration. Confirms
our flange convention matches the canonical URDF; the fastwam copy (tool0 =
fingertip) is the older snapshot.

Co-Authored-By: Claude Opus 4.8 <noreply@anthropic.com>

File: urdf/dk1_dual_arm.urdf (robot description, URDF)
Before this commit: robot dk1_dual_arm, 28 links, 27 joints
Joints:
- removed joint left_gripper_tool0
- removed joint right_gripper_tool0
- added joint left_tool0_joint: type fixed, parent left_link6-7, child left_tool0, origin xyz=0 0 0 rpy=-1.5707963267948966 0 -1.5707963267948966
- added joint right_tool0_joint: type fixed, parent right_link6-7, child right_tool0, origin xyz=0 0 0 rpy=-1.5707963267948966 0 -1.5707963267948966
